File: bluetooth_speaker.kicad_sch (KiCad schematic)
At the start: 22 parts, among them U1 MAX98357A, U2 XL4015, U3 ESP32-WROOM-32UE

Commit message: Updated files to work on
Parts:
- removed C3, C7: 1µF, symbol Device:C_Small
- removed C4: 330µF/25V, symbol Device:C_Small_US
- removed C8: 220µF/50V, symbol Device:C_Small_US
- removed L1: 47µH/5A, symbol Device:L
- removed R1: 300kΩ, symbol Device:R_US
- removed R2: 16.5kΩ, symbol Device:R_US
- removed R3, R4, R5: 10kΩ, symbol Device:R_US
- added C12: 12pF, symbol Device:C_Small
- added C13: 10µF, Capacitor_SMD:C_0603_1608Metric_Pad1.08x0.95mm_HandSolder, symbol Device:C_Small
- added C3: EEEHA1E331P, EEE_HA1E331P:CAP_EEEHA1E331P, symbol EEEHA1E331P:EEEHA1E331P
- added C4: 33nF, Capacitor_SMD:C_0603_1608Metric_Pad1.08x0.95mm_HandSolder, symbol Device:C_Small
- added C7: EEETK1H221AQ, EEETK1H221AQ:CAP_EEETK1H221AQ, symbol EEETK1H221AQ:EEETK1H221AQ
- added C8: 22µF, Capacitor_SMD:C_0603_1608Metric_Pad1.08x0.95mm_HandSolder, symbol Device:C_Small
- added L1: SDR2207-470KL, footprints:IND_BOURNS_SDR2207, symbol 2025-11-03_09-40-57:SDR2207-470KL
- added R1: 300kΩ, Resistor_SMD:R_0603_1608Metric_Pad0.98x0.95mm_HandSolder, symbol Device:R_Small_US
- added R2, R3, R5: 10kΩ, Resistor_SMD:R_0603_1608Metric_Pad0.98x0.95mm_HandSolder, symbol Device:R_Small_US
- added R4, R7: 0Ω, Resistor_SMD:R_0603_1608Metric_Pad0.98x0.95mm_HandSolder, symbol Device:R_Small_US
- added R6: 5.05MΩ, Resistor_SMD:R_0603_1608Metric_Pad0.98x0.95mm_HandSolder, symbol Device:R_Small_US
- added R8: 16.5kΩ, Resistor_SMD:R_0603_1608Metric_Pad0.98x0.95mm_HandSolder, symbol Device:R_Small_US
- added Y2: ABS07-166-32.768KHZ-T, ABS07-166-32.768KHZ-T:XTAL_ABS07-166-32.768KHZ-T, symbol ABS07-166-32.768KHZ-T:ABS07-166-32.768KHZ-T
- C1: value 10µF -> 0.1µF; footprint (none) -> Capacitor_SMD:C_0603_1608Metric_Pad1.08x0.95mm_HandSolder
- C10, C6, C9: footprint (none) -> Capacitor_SMD:C_0603_1608Metric_Pad1.08x0.95mm_HandSolder
- C11: value 1µF -> 12pF
- C2: value 0.1µF -> 1µF; footprint (none) -> Capacitor_SMD:C_0603_1608Metric_Pad1.08x0.95mm_HandSolder
- C5: value 33nF -> 1µF; footprint (none) -> Capacitor_SMD:C_0603_1608Metric_Pad1.08x0.95mm_HandSolder
Connections:
- net GNDREF: now also C6.2, C12.2, C13.2, C3.2, C7.2, C8.2, R2.1
- net SD_MODE: now also R1.1
- net at U3.27 (IO16): now also R5.2
- net at C5.2: now also U2.4 (VC); no longer U2.2 (FB)
- net at D2.1 (K), U2.3 (SW): now also L1.2
- net at C11.1: now also R6.2, R7.1, Y2.1; no longer U3.3 (EN)
- net at U3.8 (IO32): now also R4.2
- net at U3.9 (IO33): now also R7.2
- net at U1.4 (~{SD_MODE}): now also R1.2
- net Vdd renamed Vdd_5V
- net Vdd_5V: now also C5.1, C7.1
- net Vdd33 renamed Vdd_3.3V
- net Vdd_3.3V: now also C13.1, C3.1, C4.1, C8.1, L1.1, R3.2, R5.1, R8.2; no longer C10.1, C5.1
- new net: C4.2, R2.2, R8.1, U2.2 (FB)
- new net: C10.1, R3.1, U3.3 (EN)
- new net: C12.1, R4.1, R6.1, Y2.2
- no-connect marks 22 -> 20
