File: bluetooth_speaker/bluetooth_speaker.kicad_sch (KiCad schematic)
At the start: 23 parts, among them J1 Conn_Coaxial, J2 USB_C_Receptacle_USB2.0_16P, J3 282836-4, J5 Conn_01x04_Pin, U4 ESP32-D0WD-V3, Y1 40MHz(±10 ppm)

Commit message: Updated PCB traces
Parts:
- C16: footprint SamacSys_Parts:GRM033D70J224ME01D -> SamacSys_Parts:CAPC3216X94N
- C17: footprint SamacSys_Parts:GRM033D70J224ME01D -> SamacSys_Parts:CAPC3216X170N
- L3: footprint SamacSys_Parts:LQP03TG3N1B02D -> SamacSys_Parts:LQW2BAN11NG00L
Changed lines of the file:
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@@
 			)
 		)
-		(property "Footprint" "SamacSys_Parts:GRM033D70J224ME01D"
+		(property "Footprint" "SamacSys_Parts:CAPC3216X170N"
 			(at 242.57 137.16 0)
 			(effects
@@
 			)
 		)
-		(property "Footprint" "SamacSys_Parts:LQP03TG3N1B02D"
+		(property "Footprint" "SamacSys_Parts:LQW2BAN11NG00L"
 			(at 232.41 133.35 0)
 			(effects
@@
 			)
 		)
-		(property "Datasheet" "https://www.mouser.pl/datasheet/3/76/2/JELF243C_0015.pdf"
+		(property "Datasheet" "https://www.mouser.pl/ProductDetail/Murata-Electronics/LQW2BAS2N7J00L?qs=rkhjVJ6%2F3EIoAem%252BmvnZ5w%3D%3D"
 			(at 232.41 133.35 0)
 			(effects
@@
 			)
 		)
-		(property "Footprint" "SamacSys_Parts:GRM033D70J224ME01D"
+		(property "Footprint" "SamacSys_Parts:CAPC3216X94N"
 			(at 222.25 137.16 0)
 			(effects

Commit message: Completed the PCB design
Connections:
- net BCLK: now also U4.36 (GPIO23); no longer U4.15 (GPIO26)
- net BTN_PLAY: now also U4.16 (GPIO27); no longer U4.36 (GPIO23)
- net BTN_VOL_DOWN: now also U4.14 (GPIO25); no longer U4.34 (GPIO5)
- net BTN_VOL_UP: now also U4.15 (GPIO26); no longer U4.35 (GPIO18)
- net DATA: now also U4.35 (GPIO18); no longer U4.39 (GPIO22)
- net LRCLK: now also U4.39 (GPIO22); no longer U4.14 (GPIO25)
- net SD_MODE: now also U4.34 (GPIO5); no longer U4.16 (GPIO27)
Other:
- note added: "MUSIC CONTROL CONN"
- company: (none) -> Politechnika Poznańska
- title: (none) -> bluetooth speaker
- moved on the sheet: J5
Changed lines of the file:
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@@
 	(generator_version "9.0")
 	(paper "A4")
+	(title_block
+		(title "bluetooth speaker")
+		(date "2026-01-05")
+		(rev "1.0")
+		(company "Politechnika Poznańska")
+	)
 	(text "CRYSTAL"
 		(exclude_from_sim no)
@@
 		)
 	)
+	(text "MUSIC CONTROL CONN"
+		(exclude_from_sim no)
+		(at 135.89 165.862 0)
+		(effects
+			(font
+				(size 1.27 1.27)
+			)
+		)
+	)
 	(junction
 		(at 43.18 39.37)
@@
 	(wire
 		(pts
-			(xy 135.89 185.42) (xy 146.05 185.42)
+			(xy 133.35 187.96) (xy 143.51 187.96)
 		)
 		(stroke
@@
 		)
 	)
+	(polyline
+		(pts
+			(xy 194.31 163.83) (xy 194.31 165.1)
+		)
+		(stroke
+			(width 0)
+			(type dash)
+		)
+	)
 	(wire
 		(pts
@@
 	(wire
 		(pts
-			(xy 144.78 182.88) (xy 146.05 182.88)
+			(xy 142.24 185.42) (xy 143.51 185.42)
 		)
 		(stroke
@@
 		)
 	)
+	(polyline
+		(pts
+			(xy 106.68 158.75) (xy 194.31 158.75)
+		)
+		(stroke
+			(width 0)
+			(type dash)
+		)
+	)
 	(wire
 		(pts
@@
 	(wire
 		(pts
-			(xy 144.78 180.34) (xy 146.05 180.34)
+			(xy 142.24 182.88) (xy 143.51 182.88)
 		)
 		(stroke
@@
 	(wire
 		(pts
-			(xy 144.78 177.8) (xy 146.05 177.8)
+			(xy 142.24 180.34) (xy 143.51 180.34)
 		)
 		(stroke
@@
 		)
 	)
-	(label "BTN_PLAY"
+	(label "BCLK"
 		(at 137.16 64.77 0)
 		(effects
@@
 	)
 	(label "BTN_VOL_UP"
-		(at 144.78 180.34 180)
+		(at 142.24 182.88 180)
 		(effects
 			(font
@@
 		)
 	)
-	(label "BTN_VOL_UP"
+	(label "DATA"
 		(at 137.16 67.31 0)
 		(effects
@@
 	)
 	(label "BTN_PLAY"
-		(at 144.78 177.8 180)
+		(at 142.24 180.34 180)
 		(effects
 			(font
@@
 		)
 	)
-	(label "BTN_VOL_DOWN"
+	(label "SD_MODE"
 		(at 137.16 69.85 0)
 		(effects
@@
 		)
 	)
-	(label "SD_MODE"
+	(label "BTN_PLAY"
 		(at 68.58 69.85 180)
 		(effects
@@
 		)
 	)
-	(label "BCLK"
+	(label "BTN_VOL_UP"
 		(at 68.58 67.31 180)
 		(effects
@@
 	)
 	(label "BTN_VOL_DOWN"
-		(at 144.78 182.88 180)
+		(at 142.24 185.42 180)
 		(effects
 			(font
@@
 		)
 	)
-	(label "DATA"
+	(label "LRCLK"
 		(at 137.16 57.15 0)
 		(effects
@@
 		)
 	)
-	(label "LRCLK"
+	(label "BTN_VOL_DOWN"
 		(at 68.58 64.77 180)
 		(effects
@@
 	(symbol
 		(lib_id "power:GND")
-		(at 135.89 185.42 270)
+		(at 133.35 187.96 270)
 		(unit 1)
 		(exclude_from_sim no)
@@
 		(fields_autoplaced yes)
 		(property "Reference" "#PWR047"
-			(at 129.54 185.42 0)
+			(at 127 187.96 0)
 			(effects
 				(font
@@
 		)
 		(property "Value" "GND"
-			(at 130.81 185.42 0)
+			(at 128.27 187.96 0)
 			(effects
 				(font
@@
 		)
 		(property "Footprint" ""
-			(at 135.89 185.42 0)
+			(at 133.35 187.96 0)
 			(effects
 				(font
@@
 		)
 		(property "Datasheet" ""
-			(at 135.89 185.42 0)
+			(at 133.35 187.96 0)
 			(effects
 				(font
@@
 		)
 		(property "Description" "Power symbol creates a global label with name \"GND\" , ground"
-			(at 135.89 185.42 0)
+			(at 133.35 187.96 0)
 			(effects
 				(font
@@
 	(symbol
 		(lib_id "Connector:Conn_01x04_Pin")
-		(at 151.13 182.88 180)
+		(at 148.59 185.42 180)
 		(unit 1)
 		(exclude_from_sim no)
@@
 		(dnp no)
 		(property "Reference" "J5"
-			(at 152.654 173.228 0)
+			(at 150.114 175.768 0)
 			(effects
 				(font
@@
 		)
 		(property "Value" "Conn_01x04_Pin"
-			(at 152.654 170.688 0)
+			(at 150.114 173.228 0)
 			(effects
 				(font
@@
 		)
 		(property "Footprint" "Connector_JST:JST_PH_B4B-PH-K_1x04_P2.00mm_Vertical"
-			(at 151.13 182.88 0)
+			(at 148.59 185.42 0)
 			(effects
 				(font
@@
 		)
 		(property "Datasheet" "~"
-			(at 151.13 182.88 0)
+			(at 148.59 185.42 0)
 			(effects
 				(font
@@
 		)
 		(property "Description" "Generic connector, single row, 01x04, script generated"
-			(at 151.13 182.88 0)
+			(at 148.59 185.42 0)
 			(effects
 				(font

Commit message: Exchanged CP2102N to CP2102C due to discontinuation
Parts:
- C10, C12, C15, C5: value 0.1µF -> 0.1uF
- C13: value 10µF -> 10uF
- C14, C18, C9: value 1µF -> 1uF
- C17: footprint SamacSys_Parts:CAPC3216X170N -> SamacSys_Parts:CAPC3216X94N
Changed lines of the file:
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@@
 			)
 		)
-		(property "Footprint" "SamacSys_Parts:CAPC3216X170N"
+		(property "Footprint" "SamacSys_Parts:CAPC3216X94N"
 			(at 242.57 137.16 0)
 			(effects
@@
 			)
 		)
-		(property "Value" "10µF"
+		(property "Value" "10uF"
 			(at 14.732 44.196 0)
 			(effects
@@
 			)
 		)
-		(property "Value" "0.1µF"
+		(property "Value" "0.1uF"
 			(at 36.322 82.296 0)
 			(effects
@@
 			)
 		)
-		(property "Value" "0.1µF"
+		(property "Value" "0.1uF"
 			(at 36.322 44.196 0)
 			(effects
@@
 			)
 		)
-		(property "Value" "1µF"
+		(property "Value" "1uF"
 			(at 153.162 44.196 0)
 			(effects
@@
 			)
 		)
-		(property "Value" "0.1µF"
+		(property "Value" "0.1uF"
 			(at 151.892 67.056 0)
 			(effects
@@
 			)
 		)
-		(property "Value" "1µF"
+		(property "Value" "1uF"
 			(at 151.892 94.996 0)
 			(effects
@@
 			)
 		)
-		(property "Value" "0.1µF"
+		(property "Value" "0.1uF"
 			(at 35.052 28.956 0)
 			(effects
@@
 			)
 		)
-		(property "Value" "1µF"
+		(property "Value" "1uF"
 			(at 24.892 44.196 0)
 			(effects

Commit message: Updated crystal design
Parts:
- Y1: footprint Crystal:Crystal_SMD_SeikoEpson_MC306-4Pin_8.0x3.2mm -> SamacSys_Parts:FW400WFMR1
Changed lines of the file:
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@@
 			)
 		)
-		(property "Footprint" "Crystal:Crystal_SMD_SeikoEpson_MC306-4Pin_8.0x3.2mm"
+		(property "Footprint" "SamacSys_Parts:FW400WFMR1"
 			(at 168.91 132.08 0)
 			(effects
